Commit message: Add GPS sensor integration and configuration to Asinus robot model

File: asinus_gz/urdf/asinus_gz.xacro (robot description, xacro)
@@ -12,4 +12,5 @@
   <xacro:include filename="$(find ${package_name})/urdf/include/ros2_control_macro.urdf.xacro" />
   <xacro:include filename="$(find ${package_name})/urdf/include/sensors/kinect.urdf.xacro" />
+  <xacro:include filename="$(find ${package_name})/urdf/include/sensors/gps.urdf.xacro" />
   <xacro:arg name="yaml_config_dir" default="$(find ${package_name})/config/${robot_name}" />
   <xacro:property name="caster_wheel_yaml" value="$(arg yaml_config_dir)/caster_wheel.yaml" />
@@ -104,11 +105,4 @@
     <origin xyz="-0.033 -0.010 0.02" rpy="3.1416 0 0"/>
   </joint>
-  <!-- GPS link -->
-  <link name="gps_link"/>
-  <joint name="gps_joint" type="fixed">
-    <parent link="base_link"/>
-    <child link="gps_link"/>
-    <origin xyz="0 0 0.05" rpy="0 0 0"/>
-  </joint>
    <xacro:if value="$(arg use_gazebo_ros_control)">
     <ros2_control name="GazeboSimSystem" type="system">
@@ -169,15 +163,4 @@
   </gazebo>
   <!-- GPS Sensor -->
-  <gazebo reference="gps_link">
-    <sensor name="navsat" type="navsat">
-      <always_on>1</always_on>
-      <update_rate>1</update_rate>
-      <topic>navsat</topic>
-      <navsat>
-        <position_sensing>
-        </position_sensing>
-      </navsat>
-    </sensor>
-  </gazebo>
   </xacro:if>
   <xacro:unless value="$(arg use_gazebo_ros_control)">
@@ -188,3 +171,5 @@
   <!-- Kinect Sensor -->
   <xacro:sensor_kinect parent="base_link" namespace="$(arg namespace)"/>
+  <!-- GPS Sensor -->
+  <xacro:sensor_gps parent="base_link" namespace="$(arg namespace)"/>
 </robot>
