Commit message: Add RoboCup 2014 SPL Field model configuration and SDF definition
- Created model.config for the RoboCup 2014 SPL Field with metadata including name, version, author, and description.
- Added model.sdf file defining the static field model with visual and collision elements, including sidelines, endlines, halfway line, area lines, penalty spots, and center circle.
- Configured materials and poses for each visual element to accurately represent the field layout according to the 2014 rules.

File: asinus_description/urdf/asinus.urdf.xacro (robot description, xacro)
@@ -107,4 +107,11 @@
     <origin xyz="-0.033 -0.010 0.02" rpy="3.1416 0 0"/>
   </joint>
+  <!-- GPS link -->
+  <link name="gps_link"/>
+  <joint name="gps_joint" type="fixed">
+    <parent link="base_link"/>
+    <child link="gps_link"/>
+    <origin xyz="-0.033 -0.010 0.02" rpy="3.1416 0 0"/>
+  </joint>
   <!-- ROS2 Control -->
   <xacro:ros2_control_macro robot_prefix="" />

File: asinus_description/urdf/include/sensors/kinect.urdf.xacro (robot description, xacro)
@@ -13,49 +13,22 @@
     <gazebo reference="camera_link">
       <!-- RGB Camera Sensor -->
-      <sensor name="kinect_camera" type="camera">
-        <always_on>true</always_on>
-        <visualize>true</visualize>
-        <update_rate>30</update_rate>
-        <topic>camera/image_raw</topic>
-        <gz_frame_id>camera_rgb_optical_frame</gz_frame_id>
-        <camera name="kinect_camera">
-          <camera_info_topic>camera/camera_info</camera_info_topic>
-          <horizontal_fov>1.3962634</horizontal_fov>
+      <sensor name="rgbd_camera" type="rgbd_camera">
+        <camera>
+          <horizontal_fov>${60.0*M_PI/180.0}</horizontal_fov>
           <image>
+            <format>B8G8R8</format>
             <width>640</width>
             <height>480</height>
-            <format>R8G8B8</format>
           </image>
           <clip>
-            <near>0.02</near>
-            <far>300</far>
+            <near>0.05</near>
+            <far>8.0</far>
           </clip>
-          <noise>
-            <type>gaussian</type>
-            <mean>0.0</mean>
-            <stddev>0.007</stddev>
-          </noise>
         </camera>
-      </sensor>
-      <!-- Depth Camera Sensor -->
-      <sensor name="kinect_depth" type="depth_camera">
         <always_on>true</always_on>
+        <update_rate>20.0</update_rate>
         <visualize>true</visualize>
-        <update_rate>15</update_rate>
-        <topic>camera/depth/image_raw</topic>
-        <gz_frame_id>camera_depth_optical_frame</gz_frame_id>
-        <depth_camera name="kinect_depth">
-          <camera_info_topic>camera/depth/camera_info</camera_info_topic>
-          <horizontal_fov>1.047</horizontal_fov>
-          <image>
-            <width>640</width>
-            <height>480</height>
-            <format>FLOAT32</format>
-          </image>
-          <clip>
-            <near>0.1</near>
-            <far>10.0</far>
-          </clip>
-        </depth_camera>
+        <topic>rgbd_camera</topic>
+        <enable_metrics>true</enable_metrics>
       </sensor>
     </gazebo>

File: asinus_gz/urdf/asinus_gz.xacro (robot description, xacro)
@@ -104,4 +104,11 @@
     <origin xyz="-0.033 -0.010 0.02" rpy="3.1416 0 0"/>
   </joint>
+  <!-- GPS link -->
+  <link name="gps_link"/>
+  <joint name="gps_joint" type="fixed">
+    <parent link="base_link"/>
+    <child link="gps_link"/>
+    <origin xyz="0 0 0.05" rpy="0 0 0"/>
+  </joint>
    <xacro:if value="$(arg use_gazebo_ros_control)">
     <ros2_control name="GazeboSimSystem" type="system">
@@ -144,53 +151,36 @@
   <gazebo>
     <plugin filename="gz_ros2_control-system" name="gz_ros2_control::GazeboSimROS2ControlPlugin">
-      <ros>
-        <namespace>$(arg namespace)</namespace>
-      </ros>
       <parameters>$(find ros2_control_asinus)/config/diffbot_controllers.yaml</parameters>
     </plugin>
+    <!-- Linear Battery Plugin -->
+    <!-- TODO calibration -->
+    <plugin filename="gz-sim-linearbatteryplugin-system"
+            name="gz::sim::systems::LinearBatteryPlugin">
+          <battery_name>linear_battery</battery_name>
+          <voltage>24.00</voltage>
+          <open_circuit_voltage_constant_coef>24.00</open_circuit_voltage_constant_coef>
+          <capacity>105.5</capacity>
+          <power_load>700.0</power_load>
+          <fix_issue_225>true</fix_issue_225>
+          <enable_recharge>true</enable_recharge>
+          <charging_time>3.0</charging_time>
+          <recharge_by_topic>true</recharge_by_topic>
+    </plugin>
+  </gazebo>
+  <!-- GPS Sensor -->
+  <gazebo reference="gps_link">
+    <sensor name="navsat" type="navsat">
+      <always_on>1</always_on>
+      <update_rate>1</update_rate>
+      <topic>navsat</topic>
+      <navsat>
+        <position_sensing>
+        </position_sensing>
+      </navsat>
+    </sensor>
   </gazebo>
   </xacro:if>
   <xacro:unless value="$(arg use_gazebo_ros_control)">
 	  <gazebo>
-    <plugin name="ignition::gazebo::systems::JointStatePublisher" filename="ignition-gazebo-joint-state-publisher-system">
-      <ros>
-        <namespace>${robot_namespace}</namespace>
-        <remapping>~/out:=joint_states</remapping>
-        <remapping>/tf:=tf</remapping>
-      </ros>
-      <update_rate>30</update_rate>
-      <joint_name>right1_motor_hub_joint</joint_name>
-      <joint_name>right2_motor_hub_joint</joint_name>
-      <joint_name>left1_motor_hub_joint</joint_name>
-      <joint_name>left2_motor_hub_joint</joint_name>
-    </plugin>
-    <plugin filename="gz_ros2_control-system" name="gz_ros2_control::GazeboSimROS2ControlPlugin">
-      <ros>
-        <namespace>${robot_namespace}</namespace>
-        <remapping>/odom:=odom</remapping>
-        <remapping>/tf:=tf</remapping>
-      </ros>
-      <!-- wheels -->
-      <left_joint>left1_motor_hub_joint</left_joint>
-      <right_joint>right1_motor_hub_joint</right_joint>
-      <left2_joint>left2_motor_hub_joint</left2_joint>
-      <right2_joint>right2_motor_hub_joint</right2_joint>
-      <!-- kinematics -->
-      <wheel_separation>0.567</wheel_separation>
-      <wheel_radius>0.079</wheel_radius>
-      <!-- limits -->
-      <max_wheel_torque>20</max_wheel_torque>
-      <max_wheel_acceleration>2</max_wheel_acceleration>
-      <!-- output -->
-      <publish_odom>true</publish_odom>
-      <publish_odom_tf>true</publish_odom_tf>
-      <odometry_frame>odom</odometry_frame>
-      <robot_base_frame>base_link</robot_base_frame>
-    </plugin>
-    <plugin  filename="gz-sim-sensors-system"  name="gz::sim::systems::Sensors">
-      <render_engine>ogre2</render_engine>
-    </plugin>
-    <plugin  filename="gz-sim-imu-system"  name="gz::sim::systems::Imu">
-    </plugin>
     </gazebo>
   </xacro:unless>

Commit message: feat: Add Asinus SLAM package with optimized RTABMap configuration
- Created `asinus_slam` package for SLAM functionality using RTABMap, EKF, LIDAR, and GPS.
- Implemented optimized topic subscriptions in `rtabmap_optimized.yaml` to reduce unnecessary sensor data processing.
- Developed launch files for SLAM and simulation, including `slam.launch.py` and `asinus_slam_sim.launch.py`.
- Added configuration files for EKF and RTABMap to enhance performance and reduce CPU/memory usage.
- Included necessary dependencies in `CMakeLists.txt` and `package.xml`.
- Documented optimization strategies and configurations in `README_optimization.md`.
- Introduced a new world model in `farm.sdf` for simulation purposes.

File: asinus_description/urdf/asinus.urdf.xacro (robot description, xacro)
@@ -98,5 +98,5 @@
     <parent link="base_link"/>
     <child link="odom_link"/>
-    <origin xyz="0 0 0" rpy="0 0 3.1416"/>
+    <origin xyz="0 0 0" rpy="0 0 0"/>
   </joint>
   <!-- MPU link -->

File: asinus_description/urdf/include/sensors/gps.urdf.xacro (robot description, xacro)
@@ -13,4 +13,5 @@
     <gazebo reference="gps_link">
       <!-- GPS Sensor -->
+      <gz_frame_id>gps_link</gz_frame_id>
       <sensor name="navsat_sensor" type="navsat">
           <always_on>1</always_on>

File: asinus_description/urdf/include/sensors/imu.urdf.xacro (robot description, xacro)
@@ -1 +1,119 @@
-<
+<?xml version="1.0"?>
+<robot name="sensor_imu" xmlns:xacro="http://www.ros.org/wiki/xacro">
+  <!-- Define pi constant -->
+  <xacro:property name="M_PI" value="3.14159265359"/>
+  <xacro:property name="imu_px" value="-0.033" />
+  <xacro:property name="imu_py" value="-0.010" />
+  <xacro:property name="imu_pz" value="0.2" />
+  <xacro:property name="imu_or" value="0" />
+  <xacro:property name="imu_op" value="0" />
+  <xacro:property name="imu_oy" value="0" />
+  <!-- IMU for simulation -->
+  <xacro:macro name="asinus_imu" params="namespace:=''">
+    <gazebo reference="imu_link">
+      <!-- IMU Sensor -->
+      <sensor name="imu_sensor" type="imu">
+          <always_on>1</always_on>
+          <update_rate>20</update_rate>
+          <topic>imu</topic>
+          <gz_frame_id>imu_link</gz_frame_id>
+          <imu>
+            <angular_velocity>
+              <x>
+                <noise type="gaussian">
+                  <mean>0.0</mean>
+                  <stddev>0.0</stddev>
+                </noise>
+              </x>
+              <y>
+                <noise type="gaussian">
+                  <mean>0.0</mean>
+                  <stddev>0.0</stddev>
+                </noise>
+              </y>
+              <z>
+                <noise type="gaussian">
+                  <mean>0.0</mean>
+                  <stddev>0.0</stddev>
+                </noise>
+              </z>
+            </angular_velocity>
+            <linear_acceleration>
+              <x>
+                <noise type="gaussian">
+                  <mean>0.0</mean>
+                  <stddev>0.0</stddev>
+                </noise>
+              </x>
+              <y>
+                <noise type="gaussian">
+                  <mean>0.0</mean>
+                  <stddev>0.0</stddev>
+                </noise>
+              </y>
+              <z>
+                <noise type="gaussian">
+                  <mean>0.0</mean>
+                  <stddev>0.0</stddev>
+                </noise>
+              </z>
+            </linear_acceleration>
+          </imu>
+    </sensor>
+        <sensor name="magnetometer" type="magnetometer">
+            <always_on>1</always_on>
+            <update_rate>20</update_rate>
+            <visualize>true</visualize>
+            <topic>magnetometer</topic>
+            <enable_metrics>true</enable_metrics>
+            <magnetometer>
+            <x>
+                <noise type="gaussian">
+                <mean>0.0</mean>
+                <stddev>0.0</stddev>
+                </noise>
+            </x>
+            <y>
+                <noise type="gaussian">
+                <mean>0.0</mean>
+                <stddev>0.0</stddev>
+                </noise>
+            </y>
+            <z>
+                <noise type="gaussian">
+                <mean>0.0</mean>
+                <stddev>0.0</stddev>
+                </noise>
+            </z>
+            </magnetometer>
+    </sensor>
+    </gazebo>
+  </xacro:macro>
+  <!-- IMU Sensor Macro -->
+  <xacro:macro name="sensor_imu" params="parent namespace:=''">
+    <joint name="imu_joint" type="fixed">
+      <origin xyz="${imu_px} ${imu_py} ${imu_pz}" rpy="${imu_or} ${imu_op} ${imu_oy}"/>
+      <parent link="${parent}"/>
+      <child link="imu_link" />
+    </joint>
+    <link name="imu_link">
+      <visual>
+        <origin xyz="0 0 0" rpy="0 0 0"/>
+        <geometry>
+          <box size="0.02 0.015 0.005"/>
+        </geometry>
+        <material name="imu_material">
+          <color rgba="0.1 0.1 0.8 1.0"/>
+        </material>
+      </visual>
+      <collision>
+        <origin xyz="0 0 0" rpy="0 0 0"/>
+        <geometry>
+          <box size="0.02 0.015 0.005"/>
+        </geometry>
+      </collision>
+    </link>
+    <!-- IMU sensor for simulation -->
+    <xacro:asinus_imu namespace="${namespace}"/>
+  </xacro:macro>
+</robot>

File: asinus_description/urdf/include/sensors/kinect.urdf.xacro (robot description, xacro)
@@ -5,5 +5,5 @@
   <xacro:property name="cam_px" value="-0.087" />
   <xacro:property name="cam_py" value="-0.0125" />
-	<xacro:property name="cam_pz" value="0.2870" />
+	<xacro:property name="cam_pz" value="0.6" />
 	<xacro:property name="cam_or" value="0" />
 	<xacro:property name="cam_op" value="0" />
@@ -13,9 +13,8 @@
     <gazebo reference="camera_link">
       <!-- RGB Camera Sensor -->
-      <sensor name="rgbd_camera" type="rgbd_camera">
+      <sensor name="rgb_camera" type="camera">
         <camera>
           <horizontal_fov>${60.0*M_PI/180.0}</horizontal_fov>
           <image>
-            <format>B8G8R8</format>
             <width>640</width>
             <height>480</height>
@@ -23,5 +22,5 @@
           <clip>
             <near>0.05</near>
-            <far>8.0</far>
+            <far>100.0</far>
           </clip>
         </camera>
@@ -29,6 +28,28 @@
         <update_rate>20.0</update_rate>
         <visualize>true</visualize>
-        <topic>rgbd_camera</topic>
+        <topic>kinect_rgb/image</topic>
+        <gz_frame_id>camera_rgb_optical_frame</gz_frame_id>
         <enable_metrics>true</enable_metrics>
+      </sensor>
+    </gazebo>
+    <gazebo reference="camera_depth_frame">
+      <!-- Depth Camera Sensor -->
+      <sensor name="depth_camera" type="depth">
+        <update_rate>20.0</update_rate>
+        <topic>kinect_depth/image</topic>
+        <gz_frame_id>camera_depth_optical_frame</gz_frame_id>
+        <horizontal_fov>${60.0*M_PI/180.0}</horizontal_fov>
+        <enable_metrics>true</enable_metrics>
+        <depth>
+          <clip>
+            <near>0.05</near>
+            <far>8.0</far>
+          </clip>
+          <image>
+            <format>R32F</format>
+            <width>640</width>
+            <height>480</height>
+          </image>
+        </depth>
       </sensor>
     </gazebo>
@@ -43,5 +64,5 @@
     <link name="camera_rgb_frame"/>
     <joint name="camera_rgb_optical_joint" type="fixed">
-      <origin xyz="0 0 0" rpy="${-M_PI/2} 0 ${-M_PI/2}" />
+      <origin xyz="0 0 0" rpy="${-M_PI/2} 0 ${3*M_PI/2}"/>
       <parent link="camera_rgb_frame" />
       <child link="camera_rgb_optical_frame" />
@@ -53,5 +74,5 @@
       <child link="camera_link"/>
     </joint>
-      <link name="camera_link">
+    <link name="camera_link">
       <visual>
        <origin xyz="0 0 0" rpy="0 0 ${M_PI/2}"/>
@@ -74,16 +95,16 @@
       </inertial>
     </link>
-	<joint name="camera_depth_joint" type="fixed">
-	  <origin xyz="0 ${2 * -cam_py} 0" rpy="0 0 0" />
-	  <parent link="camera_rgb_frame" />
-	  <child link="camera_depth_frame" />
-	</joint>
-	<link name="camera_depth_frame"/>
-	<joint name="camera_depth_optical_joint" type="fixed">
-	  <origin xyz="0 0 0" rpy="${-M_PI/2} 0 ${-M_PI/2}" />
-	  <parent link="camera_depth_frame" />
-	  <child link="camera_depth_optical_frame" />
-	</joint>
-	<link name="camera_depth_optical_frame"/>
+    <joint name="camera_depth_joint" type="fixed">
+      <origin xyz="${cam_px} ${2 * -cam_py} ${cam_pz}" rpy="${cam_or} ${cam_op} ${cam_oy}"/>
+      <parent link="camera_rgb_frame" />
+      <child link="camera_depth_frame" />
+    </joint>
+    <link name="camera_depth_frame"/>
+    <joint name="camera_depth_optical_joint" type="fixed">
+      <origin xyz="0 0 0" rpy="${-M_PI/2} 0 ${3*M_PI/2}" />
+      <parent link="camera_depth_frame" />
+      <child link="camera_depth_optical_frame" />
+    </joint>
+    <link name="camera_depth_optical_frame"/>
 	<!-- Kinect sensor for simulation -->
 	<xacro:asinus_kinect namespace="${namespace}"/>

File: asinus_gz/urdf/asinus_gz.xacro (robot description, xacro)
@@ -13,4 +13,6 @@
   <xacro:include filename="$(find ${package_name})/urdf/include/sensors/kinect.urdf.xacro" />
   <xacro:include filename="$(find ${package_name})/urdf/include/sensors/gps.urdf.xacro" />
+  <xacro:include filename="$(find ${package_name})/urdf/include/sensors/imu.urdf.xacro" />
+  <xacro:include filename="$(find ${package_name})/urdf/include/sensors/lidar.urdf.xacro" />
   <xacro:arg name="yaml_config_dir" default="$(find ${package_name})/config/${robot_name}" />
   <xacro:property name="caster_wheel_yaml" value="$(arg yaml_config_dir)/caster_wheel.yaml" />
@@ -96,12 +98,5 @@
     <parent link="base_link"/>
     <child link="odom_link"/>
-    <origin xyz="0 0 0" rpy="0 0 3.1416"/>
-  </joint>
-  <!-- MPU link -->
-  <link name="mpu_link"/>
-  <joint name="mpu_joint" type="fixed">
-    <parent link="base_link"/>
-    <child link="mpu_link"/>
-    <origin xyz="-0.033 -0.010 0.02" rpy="3.1416 0 0"/>
+    <origin xyz="0 0 0" rpy="0 0 0"/>
   </joint>
    <xacro:if value="$(arg use_gazebo_ros_control)">
@@ -112,6 +107,6 @@
     <joint name="left1_motor_hub_joint">
       <command_interface name="velocity">
-        <param name="min">-1</param>
-        <param name="max">1</param>
+        <param name="min">-3</param>
+        <param name="max">3</param>
       </command_interface>
       <state_interface name="position"/>
@@ -120,6 +115,6 @@
     <joint name="left2_motor_hub_joint">
       <command_interface name="velocity">
-        <param name="min">-1</param>
-        <param name="max">1</param>
+        <param name="min">-3</param>
+        <param name="max">3</param>
       </command_interface>
       <state_interface name="position"/>
@@ -128,6 +123,6 @@
     <joint name="right1_motor_hub_joint">
       <command_interface name="velocity">
-        <param name="min">-1</param>
-        <param name="max">1</param>
+        <param name="min">-3</param>
+        <param name="max">3</param>
       </command_interface>
       <state_interface name="position"/>
@@ -136,6 +131,6 @@
     <joint name="right2_motor_hub_joint">
       <command_interface name="velocity">
-        <param name="min">-1</param>
-        <param name="max">1</param>
+        <param name="min">-3</param>
+        <param name="max">3</param>
       </command_interface>
       <state_interface name="position"/>
@@ -173,3 +168,6 @@
   <!-- GPS Sensor -->
   <xacro:sensor_gps parent="base_link" namespace="$(arg namespace)"/>
+  <!-- IMU Sensor -->
+  <xacro:sensor_imu parent="base_link" namespace="$(arg namespace)"/>
+  <xacro:sensor_lidar parent="base_link" namespace="$(arg namespace)"/>
 </robot>
