Commit message: Refactor code structure for improved readability and maintainability

File: asinus_description/urdf/asinus.urdf.xacro (robot description, xacro)
@@ -28,12 +28,12 @@
   <xacro:property name="wheel_support_end2_yaml" value="$(arg yaml_config_dir)/wheel_support_end2.yaml" />
   <xacro:property name="wheel_support_end2_props" value="${xacro.load_yaml(wheel_support_end2_yaml)}"/>
-  <!-- Footprint link -->
-  <xacro:footprint robot_prefix=""
-                   motor_hub_props="${motor_hub_props}" />
-  <!-- Base link -->
+  <!-- Base link (must come before footprint) -->
   <xacro:base robot_prefix=""
               link_name="base_link" base_prop="${base_props}" mesh="${base_props['base']['mesh']}" >
     <origin xyz="0 0 0" rpy="0 0 ${-pi/2}" />
   </xacro:base>
+  <!-- Footprint link (after base_link is created) -->
+  <xacro:footprint robot_prefix=""
+                   motor_hub_props="${motor_hub_props}" />
   <!-- Caster Wheel -->
   <xacro:caster_wheel robot_prefix=""
@@ -90,4 +90,6 @@
   <!-- Kinect Sensor -->
   <xacro:sensor_kinect parent="base_link" namespace="$(arg frame_prefix_arg)"/>
+  <!-- IMU Sensor -->
+  <xacro:sensor_imu parent="base_link" namespace="$(arg frame_prefix_arg)"/>
   <!-- Lidar Sensor - TODO: Implement lidar sensor macros -->
   <!-- <xacro:asinus_lidar namespace="$(arg frame_prefix_arg)"/>

File: asinus_description/urdf/include/sensors/imu.urdf.xacro (robot description, xacro)
@@ -15,77 +15,9 @@
       <sensor name="imu_sensor" type="imu">
           <always_on>1</always_on>
-          <update_rate>20</update_rate>
+          <update_rate>50</update_rate>
           <topic>imu</topic>
+          <visualize>true</visualize>
           <gz_frame_id>imu_link</gz_frame_id>
-          <imu>
-            <angular_velocity>
-              <x>
-                <noise type="gaussian">
-                  <mean>0.0</mean>
-                  <stddev>0.0</stddev>
-                </noise>
-              </x>
-              <y>
-                <noise type="gaussian">
-                  <mean>0.0</mean>
-                  <stddev>0.0</stddev>
-                </noise>
-              </y>
-              <z>
-                <noise type="gaussian">
-                  <mean>0.0</mean>
-                  <stddev>0.0</stddev>
-                </noise>
-              </z>
-            </angular_velocity>
-            <linear_acceleration>
-              <x>
-                <noise type="gaussian">
-                  <mean>0.0</mean>
-                  <stddev>0.0</stddev>
-                </noise>
-              </x>
-              <y>
-                <noise type="gaussian">
-                  <mean>0.0</mean>
-                  <stddev>0.0</stddev>
-                </noise>
-              </y>
-              <z>
-                <noise type="gaussian">
-                  <mean>0.0</mean>
-                  <stddev>0.0</stddev>
-                </noise>
-              </z>
-            </linear_acceleration>
-          </imu>
-    </sensor>
-        <sensor name="magnetometer" type="magnetometer">
-            <always_on>1</always_on>
-            <update_rate>20</update_rate>
-            <visualize>true</visualize>
-            <topic>magnetometer</topic>
-            <enable_metrics>true</enable_metrics>
-            <magnetometer>
-            <x>
-                <noise type="gaussian">
-                <mean>0.0</mean>
-                <stddev>0.0</stddev>
-                </noise>
-            </x>
-            <y>
-                <noise type="gaussian">
-                <mean>0.0</mean>
-                <stddev>0.0</stddev>
-                </noise>
-            </y>
-            <z>
-                <noise type="gaussian">
-                <mean>0.0</mean>
-                <stddev>0.0</stddev>
-                </noise>
-            </z>
-            </magnetometer>
-    </sensor>
+      </sensor>
     </gazebo>
   </xacro:macro>
@@ -99,5 +31,5 @@
     <link name="imu_link">
       <visual>
-        <origin xyz="0 0 0" rpy="0 0 0"/>
+        <origin xyz="0 0 0" rpy="0  0"/>
         <geometry>
           <box size="0.02 0.015 0.005"/>

File: asinus_description/urdf/include/sensors/kinect.urdf.xacro (robot description, xacro)
@@ -78,5 +78,5 @@
        <origin xyz="0 0 0" rpy="0 0 ${M_PI/2}"/>
         <geometry>
-         <mesh filename="package:/$(find asinus_description)/meshes/sensors/kinect.dae"/>
+         <mesh filename="package:/$(find asinus_description)/meshes/${robot_name}/kinect.dae"/>
         </geometry>
       </visual>

File: asinus_gz/urdf/asinus_gz.xacro (robot description, xacro)
@@ -33,7 +33,4 @@
   <xacro:property name="wheel_support_end2_yaml" value="$(arg yaml_config_dir)/wheel_support_end2.yaml" />
   <xacro:property name="wheel_support_end2_props" value="${xacro.load_yaml(wheel_support_end2_yaml)}"/>
-  <!-- Footprint link -->
-  <xacro:footprint robot_prefix=""
-                   motor_hub_props="${motor_hub_props}" />
   <!-- Base link -->
   <xacro:base robot_prefix=""
@@ -41,4 +38,7 @@
     <origin xyz="0 0 0" rpy="0 0 ${-pi/2}" />
   </xacro:base>
+  <!-- Footprint link -->
+    <xacro:footprint robot_prefix=""
+                    motor_hub_props="${motor_hub_props}" />
   <!-- Caster Wheel -->
   <xacro:caster_wheel robot_prefix=""
@@ -103,5 +103,5 @@
     <ros2_control name="GazeboSimSystem" type="system">
     <hardware>
-      <plugin>gz_ros2_control/GazeboSimSystem</plugin>
+      <plugin>ign_ros2_control/IgnitionSystem</plugin>
     </hardware>
     <joint name="left1_motor_hub_joint">
